File: hw/MCU_Comms_Control/PwrSD.sch (KiCad schematic (older format))
At the start: 12 parts

Commit message: continue digital design
Parts:
- added C? (x2): 100nF, symbol Device:C
- added C?: 4.7uF, symbol Device:C
- added D?: 1N5819, Diode_THT:D_DO-41_SOD81_P10.16mm_Horizontal, symbol Diode:1N5819
- added U?: L7805, symbol Regulator_Linear:L7805
Connections:
- net +12V: now also C?.1, U?.1 (IN); no longer C?.1, U?.3 (VI)
- net +3.3VADC: no longer C?.1
- net +3V3: now also C?.1, C?.1
- net GND: now also C?.2, C?.2, C?.2, U?.2 (GND)
- new net: C?.1, D?.2 (A), U?.3 (OUT)
- new net +5V: C?.1, D?.1 (K), U?.3 (VI)
Other:
- note added: "12V -> 5V"
- note added: "5V → 3.3V\n"
- note added: "L78M05\nDPAK"
- note added: "SN65HVD230"
- note added: "W25Q128JVS"
- note removed: "12V → 3.3V\n(might need better thermals)"
- note removed: "SN65HVD233"
Changed lines of the file:
@@
-$EndComp
-$Comp
-L power:+12V #PWR?
-U 1 1 5FBCFFAA
-P 1300 1450
-F 0 "#PWR?" H 1300 1300 50  0001 C CNN
-F 1 "+12V" H 1315 1623 50  0000 C CNN
-F 2 "" H 1300 1450 50  0001 C CNN
-F 3 "" H 1300 1450 50  0001 C CNN
-	1    1300 1450
-	1    0    0    -1
 $EndComp
 $Comp
@@
 	1    0    0    -1
 $EndComp
-Text Notes 1500 1150 0    39   ~ 0
-12V → 3.3V\n(might need better thermals)
+Text Notes 1650 1150 0    50   ~ 0
+5V → 3.3V\n
 Wire Notes Line
 	1100 950  3150 950
@@
 $EndComp
 Text Notes 6500 1200 0    39   ~ 0
-SN65HVD233
-$Comp
-L power:+3.3VADC #PWR?
-U 1 1 5FBF6D85
+SN65HVD230
+Wire Notes Line
+	6950 1050 6950 2100
+Wire Notes Line
+	6050 2100 6050 1050
+Wire Wire Line
+	6250 1350 6250 1450
+Wire Wire Line
+	6250 1750 6250 1850
+Wire Notes Line
+	6950 2100 6050 2100
+Wire Notes Line
+	6050 1050 6950 1050
+$Comp
+L power:+3.3V #PWR?
+U 1 1 5FBC06C2
 P 6250 1350
-AR Path="/5FBF6D85" Ref="#PWR?"  Part="1"
-AR Path="/5FBC07FC/5FBF6D85" Ref="#PWR?"  Part="1"
-F 0 "#PWR?" H 6400 1300 50  0001 C CNN
-F 1 "+3.3VADC" H 6265 1523 50  0000 C CNN
+F 0 "#PWR?" H 6250 1200 50  0001 C CNN
+F 1 "+3.3V" H 6265 1523 50  0000 C CNN
 F 2 "" H 6250 1350 50  0001 C CNN
 F 3 "" H 6250 1350 50  0001 C CNN
@@
 	1    0    0    -1
 $EndComp
-Wire Notes Line
-	6950 1050 6950 2100
-Wire Notes Line
-	6050 2100 6050 1050
-Wire Wire Line
-	6250 1350 6250 1450
-Wire Wire Line
-	6250 1750 6250 1850
-Wire Notes Line
-	6950 2100 6050 2100
-Wire Notes Line
-	6050 1050 6950 1050
+$Comp
+L power:GND #PWR?
+U 1 1 5FBC1FC7
+P 7250 1850
+F 0 "#PWR?" H 7250 1600 50  0001 C CNN
+F 1 "GND" H 7255 1677 50  0000 C CNN
+F 2 "" H 7250 1850 50  0001 C CNN
+F 3 "" H 7250 1850 50  0001 C CNN
+	1    7250 1850
+	1    0    0    -1
+$EndComp
+$Comp
+L Device:C C?
+U 1 1 5FBC1FD1
+P 7250 1600
+F 0 "C?" H 7250 1700 50  0000 L CNN
+F 1 "100nF" H 7250 1500 50  0000 L CNN
+F 2 "" H 7288 1450 50  0001 C CNN
+F 3 "~" H 7250 1600 50  0001 C CNN
+	1    7250 1600
+	1    0    0    -1
+$EndComp
+Text Notes 7500 1200 0    39   ~ 0
+W25Q128JVS
+Wire Notes Line
+	7950 1050 7950 2100
+Wire Notes Line
+	7050 2100 7050 1050
+Wire Wire Line
+	7250 1350 7250 1450
+Wire Wire Line
+	7250 1750 7250 1850
+Wire Notes Line
+	7950 2100 7050 2100
+Wire Notes Line
+	7050 1050 7950 1050
+$Comp
+L power:+3.3V #PWR?
+U 1 1 5FBC1FE2
+P 7250 1350
+F 0 "#PWR?" H 7250 1200 50  0001 C CNN
+F 1 "+3.3V" H 7265 1523 50  0000 C CNN
+F 2 "" H 7250 1350 50  0001 C CNN
+F 3 "" H 7250 1350 50  0001 C CNN
+	1    7250 1350
+	1    0    0    -1
+$EndComp
+$Comp
+L power:+5V #PWR?
+U 1 1 5FBF3FE3
+P 1300 1450
+F 0 "#PWR?" H 1300 1300 50  0001 C CNN
+F 1 "+5V" H 1315 1623 50  0000 C CNN
+F 2 "" H 1300 1450 50  0001 C CNN
+F 3 "" H 1300 1450 50  0001 C CNN
+	1    1300 1450
+	1    0    0    -1
+$EndComp
+$Comp
+L Regulator_Linear:L7805 U?
+U 1 1 5FBF6864
+P 1800 2650
+F 0 "U?" H 1900 2300 50  0000 C CNN
+F 1 "L7805" H 1950 2400 50  0000 C CNN
+F 2 "" H 1825 2500 50  0001 L CIN
+F 3 "http://www.st.com/content/ccc/resource/technical/document/datasheet/41/4f/b3/b0/12/d4/47/88/CD00000444.pdf/files/CD00000444.pdf/jcr:content/translations/en.CD00000444.pdf" H 1800 2600 50  0001 C CNN
+	1    1800 2650
+	1    0    0    -1
+$EndComp
+$Comp
+L power:+12V #PWR?
+U 1 1 5FBF78E8
+P 1300 2600
+F 0 "#PWR?" H 1300 2450 50  0001 C CNN
+F 1 "+12V" H 1315 2773 50  0000 C CNN
+F 2 "" H 1300 2600 50  0001 C CNN
+F 3 "" H 1300 2600 50  0001 C CNN
+	1    1300 2600
+	1    0    0    -1
+$EndComp
+$Comp
+L Device:C C?
+U 1 1 5FBF7CAC
+P 1300 2800
+F 0 "C?" H 1300 2900 50  0000 L CNN
+F 1 "4.7uF" H 1300 2700 50  0000 L CNN
+F 2 "" H 1338 2650 50  0001 C CNN
+F 3 "~" H 1300 2800 50  0001 C CNN
+	1    1300 2800
+	1    0    0    -1
+$EndComp
+Wire Wire Line
+	1500 2650 1300 2650
+Wire Wire Line
+	1300 2650 1300 2600
+Connection ~ 1300 2650
+$Comp
+L Device:C C?
+U 1 1 5FBFB19A
+P 2200 2800
+F 0 "C?" H 2200 2900 50  0000 L CNN
+F 1 "100nF" H 2200 2700 50  0000 L CNN
+F 2 "" H 2238 2650 50  0001 C CNN
+F 3 "~" H 2200 2800 50  0001 C CNN
+	1    2200 2800
+	1    0    0    -1
+$EndComp
+Wire Wire Line
+	2200 2650 2100 2650
+$Comp
+L power:GND #PWR?
+U 1 1 5FBFC8C6
+P 1800 3100
+F 0 "#PWR?" H 1800 2850 50  0001 C CNN
+F 1 "GND" H 1805 2927 50  0000 C CNN
+F 2 "" H 1800 3100 50  0001 C CNN
+F 3 "" H 1800 3100 50  0001 C CNN
+	1    1800 3100
+	1    0    0    -1
+$EndComp
+Wire Wire Line
+	1800 2950 1800 3050
+Wire Wire Line
+	2200 2950 2200 3050
+Wire Wire Line
+	2200 3050 1800 3050
+Connection ~ 1800 3050
+Wire Wire Line
+	1800 3050 1800 3100
+Wire Wire Line
+	1800 3050 1300 3050
+Wire Wire Line
+	1300 3050 1300 2950
+Text Notes 1950 2550 2    50   ~ 0
+L78M05\nDPAK
+$Comp
+L Diode:1N5819 D?
+U 1 1 5FC007ED
+P 2450 2650
+F 0 "D?" H 2450 2433 50  0000 C CNN
+F 1 "1N5819" H 2450 2524 50  0000 C CNN
+F 2 "Diode_THT:D_DO-41_SOD81_P10.16mm_Horizontal" H 2450 2475 50  0001 C CNN
+F 3 "http://www.vishay.com/docs/88525/1n5817.pdf" H 2450 2650 50  0001 C CNN
+	1    2450 2650
+	-1   0    0    1
+$EndComp
+Wire Wire Line
+	2300 2650 2200 2650
+Connection ~ 2200 2650
+$Comp
+L power:+5V #PWR?
+U 1 1 5FC02C65
+P 2700 2600
+F 0 "#PWR?" H 2700 2450 50  0001 C CNN
+F 1 "+5V" H 2715 2773 50  0000 C CNN
+F 2 "" H 2700 2600 50  0001 C CNN
+F 3 "" H 2700 2600 50  0001 C CNN
+	1    2700 2600
+	1    0    0    -1
+$EndComp
+Wire Wire Line
+	2700 2600 2700 2650
+Wire Wire Line
+	2700 2650 2600 2650
+Wire Notes Line
+	1100 2300 3150 2300
+Wire Notes Line
+	3150 2300 3150 3350
+Wire Notes Line
+	3150 3350 1100 3350
+Wire Notes Line
+	1100 3350 1100 2300
+Text Notes 2950 3200 2    50   ~ 10
+12V -> 5V
 $EndSCHEMATC

Commit message: finish schematic of mcu/comms and start review process
Parts:
- gave numbers to parts that had none: 17
Changed lines of the file:
@@
 $EndDescr
 $Comp
-L Regulator_Linear:AMS1117-3.3 U?
+L Regulator_Linear:AMS1117-3.3 U6
 U 1 1 5FBCFFA4
 P 1800 1500
-F 0 "U?" H 1800 1742 50  0000 C CNN
+F 0 "U6" H 1800 1742 50  0000 C CNN
 F 1 "AMS1117-3.3" H 1800 1651 50  0000 C CNN
 F 2 "Package_TO_SOT_SMD:SOT-223-3_TabPin2" H 1800 1700 50  0001 C CNN
@@
 $EndComp
 $Comp
-L Device:C C?
+L Device:C C6
 U 1 1 5FBCFFB0
 P 2200 1650
-F 0 "C?" H 2315 1696 50  0000 L CNN
+F 0 "C6" H 2315 1696 50  0000 L CNN
 F 1 "22uF" H 2315 1605 50  0000 L CNN
 F 2 "" H 2238 1500 50  0001 C CNN
@@
 Tântalo
 $Comp
-L Device:C C?
+L Device:C C4
 U 1 1 5FBCFFB7
 P 1300 1650
-F 0 "C?" H 1415 1696 50  0000 L CNN
+F 0 "C4" H 1415 1696 50  0000 L CNN
 F 1 "22uF" H 1415 1605 50  0000 L CNN
 F 2 "" H 1338 1500 50  0001 C CNN
@@
 	2100 1500 2200 1500
 $Comp
-L power:GND #PWR?
+L power:GND #PWR0139
 U 1 1 5FBCFFC2
 P 1800 1900
-F 0 "#PWR?" H 1800 1650 50  0001 C CNN
+F 0 "#PWR0139" H 1800 1650 50  0001 C CNN
 F 1 "GND" H 1805 1727 50  0000 C CNN
 F 2 "" H 1800 1900 50  0001 C CNN
@@
 	2200 1850 2200 1800
 $Comp
-L power:+3.3V #PWR?
+L power:+3.3V #PWR0140
 U 1 1 5FBCFFCF
 P 2200 1450
-F 0 "#PWR?" H 2200 1300 50  0001 C CNN
+F 0 "#PWR0140" H 2200 1300 50  0001 C CNN
 F 1 "+3.3V" H 2215 1623 50  0000 C CNN
 F 2 "" H 2200 1450 50  0001 C CNN
@@
 Connection ~ 2200 1500
 $Comp
-L Device:Ferrite_Bead_Small FB?
+L Device:Ferrite_Bead_Small FB1
 U 1 1 5FBCFFD7
 P 2550 1500
-F 0 "FB?" V 2313 1500 50  0000 C CNN
+F 0 "FB1" V 2313 1500 50  0000 C CNN
 F 1 "Ferrite" V 2404 1500 50  0000 C CNN
 F 2 "" V 2480 1500 50  0001 C CNN
@@
 P 2850 1450
 AR Path="/5FBD0020" Ref="#PWR?"  Part="1"
-AR Path="/5FBC07FC/5FBD0020" Ref="#PWR?"  Part="1"
-F 0 "#PWR?" H 3000 1400 50  0001 C CNN
+AR Path="/5FBC07FC/5FBD0020" Ref="#PWR0141"  Part="1"
+F 0 "#PWR0141" H 3000 1400 50  0001 C CNN
 F 1 "+3.3VADC" H 2865 1623 50  0000 C CNN
 F 2 "" H 2850 1450 50  0001 C CNN
@@
 	2650 1500 2850 1500
 $Comp
-L power:+3.3V #PWR?
+L power:+3.3V #PWR0142
 U 1 1 5FBD670B
 P 3450 1350
-F 0 "#PWR?" H 3450 1200 50  0001 C CNN
+F 0 "#PWR0142" H 3450 1200 50  0001 C CNN
 F 1 "+3.3V" H 3465 1523 50  0000 C CNN
 F 2 "" H 3450 1350 50  0001 C CNN
@@
 $EndComp
 $Comp
-L Device:C C?
+L Device:C C8
 U 1 1 5FBD69D4
 P 3450 1600
-F 0 "C?" H 3450 1700 50  0000 L CNN
+F 0 "C8" H 3450 1700 50  0000 L CNN
 F 1 "4.7uF" H 3450 1500 50  0000 L CNN
 F 2 "" H 3488 1450 50  0001 C CNN
@@
 $EndComp
 $Comp
-L power:GND #PWR?
+L power:GND #PWR0143
 U 1 1 5FBD735F
 P 3450 1850
-F 0 "#PWR?" H 3450 1600 50  0001 C CNN
+F 0 "#PWR0143" H 3450 1600 50  0001 C CNN
 F 1 "GND" H 3455 1677 50  0000 C CNN
 F 2 "" H 3450 1850 50  0001 C CNN
@@
 	3450 1750 3450 1800
 $Comp
-L Device:C C?
+L Device:C C9
 U 1 1 5FBD96BC
 P 3700 1600
-F 0 "C?" H 3700 1700 50  0000 L CNN
+F 0 "C9" H 3700 1700 50  0000 L CNN
 F 1 "100nF" H 3700 1500 50  0000 L CNN
 F 2 "" H 3738 1450 50  0001 C CNN
@@
 $EndComp
 $Comp
-L Device:C C?
+L Device:C C10
 U 1 1 5FBD996D
 P 3950 1600
-F 0 "C?" H 3950 1700 50  0000 L CNN
+F 0 "C10" H 3950 1700 50  0000 L CNN
 F 1 "100nF" H 3950 1500 50  0000 L CNN
 F 2 "" H 3988 1450 50  0001 C CNN
@@
 $EndComp
 $Comp
-L Device:C C?
+L Device:C C11
 U 1 1 5FBD9B77
 P 4200 1600
-F 0 "C?" H 4200 1700 50  0000 L CNN
+F 0 "C11" H 4200 1700 50  0000 L CNN
 F 1 "100nF" H 4200 1500 50  0000 L CNN
 F 2 "" H 4238 1450 50  0001 C CNN
@@
 $EndComp
 $Comp
-L Device:C C?
+L Device:C C12
 U 1 1 5FBD9F85
 P 4450 1600
-F 0 "C?" H 4450 1700 50  0000 L CNN
+F 0 "C12" H 4450 1700 50  0000 L CNN
 F 1 "100nF" H 4450 1500 50  0000 L CNN
 F 2 "" H 4488 1450 50  0001 C CNN
@@
 STM32 Digital Part\n
 $Comp
-L Device:C C?
+L Device:C C13
 U 1 1 5FBDFE7D
 P 5050 1600
-F 0 "C?" H 5050 1700 50  0000 L CNN
+F 0 "C13" H 5050 1700 50  0000 L CNN
 F 1 "4.7uF" H 5050 1500 50  0000 L CNN
 F 2 "" H 5088 1450 50  0001 C CNN
@@
 $EndComp
 $Comp
-L power:GND #PWR?
+L power:GND #PWR0144
 U 1 1 5FBDFE83
 P 5050 1850
-F 0 "#PWR?" H 5050 1600 50  0001 C CNN
+F 0 "#PWR0144" H 5050 1600 50  0001 C CNN
 F 1 "GND" H 5055 1677 50  0000 C CNN
 F 2 "" H 5050 1850 50  0001 C CNN
@@
 	5300 1800 5050 1800
 $Comp
-L Device:C C?
+L Device:C C14
 U 1 1 5FBE0833
 P 5300 1600
-F 0 "C?" H 5300 1700 50  0000 L CNN
+F 0 "C14" H 5300 1700 50  0000 L CNN
 F 1 "100nF" H 5300 1500 50  0000 L CNN
 F 2 "" H 5338 1450 50  0001 C CNN
@@
 P 5050 1350
 AR Path="/5FBE216B" Ref="#PWR?"  Part="1"
-AR Path="/5FBC07FC/5FBE216B" Ref="#PWR?"  Part="1"
-F 0 "#PWR?" H 5200 1300 50  0001 C CNN
+AR Path="/5FBC07FC/5FBE216B" Ref="#PWR0145"  Part="1"
+F 0 "#PWR0145" H 5200 1300 50  0001 C CNN
 F 1 "+3.3VADC" H 5065 1523 50  0000 C CNN
 F 2 "" H 5050 1350 50  0001 C CNN
@@
 	4850 2100 4850 1050
 $Comp
-L power:GND #PWR?
+L power:GND #PWR0146
 U 1 1 5FBF6D66
 P 6250 1850
-F 0 "#PWR?" H 6250 1600 50  0001 C CNN
+F 0 "#PWR0146" H 6250 1600 50  0001 C CNN
 F 1 "GND" H 6255 1677 50  0000 C CNN
 F 2 "" H 6250 1850 50  0001 C CNN
@@
 $EndComp
 $Comp
-L Device:C C?
+L Device:C C15
 U 1 1 5FBF6D78
 P 6250 1600
-F 0 "C?" H 6250 1700 50  0000 L CNN
+F 0 "C15" H 6250 1700 50  0000 L CNN
 F 1 "100nF" H 6250 1500 50  0000 L CNN
 F 2 "" H 6288 1450 50  0001 C CNN
@@
 	6050 1050 6950 1050
 $Comp
-L power:+3.3V #PWR?
+L power:+3.3V #PWR0147
 U 1 1 5FBC06C2
 P 6250 1350
-F 0 "#PWR?" H 6250 1200 50  0001 C CNN
+F 0 "#PWR0147" H 6250 1200 50  0001 C CNN
 F 1 "+3.3V" H 6265 1523 50  0000 C CNN
 F 2 "" H 6250 1350 50  0001 C CNN
@@
 $EndComp
 $Comp
-L power:GND #PWR?
+L power:GND #PWR0148
 U 1 1 5FBC1FC7
 P 7250 1850
-F 0 "#PWR?" H 7250 1600 50  0001 C CNN
+F 0 "#PWR0148" H 7250 1600 50  0001 C CNN
 F 1 "GND" H 7255 1677 50  0000 C CNN
 F 2 "" H 7250 1850 50  0001 C CNN
@@
 $EndComp
 $Comp
-L Device:C C?
+L Device:C C16
 U 1 1 5FBC1FD1
 P 7250 1600
-F 0 "C?" H 7250 1700 50  0000 L CNN
+F 0 "C16" H 7250 1700 50  0000 L CNN
 F 1 "100nF" H 7250 1500 50  0000 L CNN
 F 2 "" H 7288 1450 50  0001 C CNN
@@
 	7050 1050 7950 1050
 $Comp
-L power:+3.3V #PWR?
+L power:+3.3V #PWR0149
 U 1 1 5FBC1FE2
 P 7250 1350
-F 0 "#PWR?" H 7250 1200 50  0001 C CNN
+F 0 "#PWR0149" H 7250 1200 50  0001 C CNN
 F 1 "+3.3V" H 7265 1523 50  0000 C CNN
 F 2 "" H 7250 1350 50  0001 C CNN
@@
 $EndComp
 $Comp
-L power:+5V #PWR?
+L power:+5V #PWR0150
 U 1 1 5FBF3FE3
 P 1300 1450
-F 0 "#PWR?" H 1300 1300 50  0001 C CNN
+F 0 "#PWR0150" H 1300 1300 50  0001 C CNN
 F 1 "+5V" H 1315 1623 50  0000 C CNN
 F 2 "" H 1300 1450 50  0001 C CNN
@@
 $EndComp
 $Comp
-L Regulator_Linear:L7805 U?
+L Regulator_Linear:L7805 U7
 U 1 1 5FBF6864
 P 1800 2650
-F 0 "U?" H 1900 2300 50  0000 C CNN
+F 0 "U7" H 1900 2300 50  0000 C CNN
 F 1 "L7805" H 1950 2400 50  0000 C CNN
 F 2 "" H 1825 2500 50  0001 L CIN
@@
 $EndComp
 $Comp
-L power:+12V #PWR?
+L power:+12V #PWR0151
 U 1 1 5FBF78E8
 P 1300 2600
-F 0 "#PWR?" H 1300 2450 50  0001 C CNN
+F 0 "#PWR0151" H 1300 2450 50  0001 C CNN
 F 1 "+12V" H 1315 2773 50  0000 C CNN
 F 2 "" H 1300 2600 50  0001 C CNN
@@
 $EndComp
 $Comp
-L Device:C C?
+L Device:C C5
 U 1 1 5FBF7CAC
 P 1300 2800
-F 0 "C?" H 1300 2900 50  0000 L CNN
+F 0 "C5" H 1300 2900 50  0000 L CNN
 F 1 "4.7uF" H 1300 2700 50  0000 L CNN
 F 2 "" H 1338 2650 50  0001 C CNN
@@
 Connection ~ 1300 2650
 $Comp
-L Device:C C?
+L Device:C C7
 U 1 1 5FBFB19A
 P 2200 2800
-F 0 "C?" H 2200 2900 50  0000 L CNN
+F 0 "C7" H 2200 2900 50  0000 L CNN
 F 1 "100nF" H 2200 2700 50  0000 L CNN
 F 2 "" H 2238 2650 50  0001 C CNN
@@
 	2200 2650 2100 2650
 $Comp
-L power:GND #PWR?
+L power:GND #PWR0152
 U 1 1 5FBFC8C6
 P 1800 3100
-F 0 "#PWR?" H 1800 2850 50  0001 C CNN
+F 0 "#PWR0152" H 1800 2850 50  0001 C CNN
 F 1 "GND" H 1805 2927 50  0000 C CNN
 F 2 "" H 1800 3100 50  0001 C CNN
@@
 L78M05\nDPAK
 $Comp
-L Diode:1N5819 D?
+L Diode:1N5819 D7
 U 1 1 5FC007ED
 P 2450 2650
-F 0 "D?" H 2450 2433 50  0000 C CNN
+F 0 "D7" H 2450 2433 50  0000 C CNN
 F 1 "1N5819" H 2450 2524 50  0000 C CNN
 F 2 "Diode_THT:D_DO-41_SOD81_P10.16mm_Horizontal" H 2450 2475 50  0001 C CNN
@@
 Connection ~ 2200 2650
 $Comp
-L power:+5V #PWR?
+L power:+5V #PWR0153
 U 1 1 5FC02C65
 P 2700 2600
-F 0 "#PWR?" H 2700 2450 50  0001 C CNN
+F 0 "#PWR0153" H 2700 2450 50  0001 C CNN
 F 1 "+5V" H 2715 2773 50  0000 C CNN
 F 2 "" H 2700 2600 50  0001 C CNN

Commit message: add footprints and lcsc code
Parts:
- C10, C11, C12, C14, C15, C16, C7, C9: footprint (none) -> Capacitor_SMD:C_0603_1608Metric; LCSC (none) -> C14663
- C13, C5, C8: footprint (none) -> Capacitor_SMD:C_0603_1608Metric; LCSC (none) -> C19666
- C4, C6: footprint (none) -> Capacitor_SMD:C_0805_2012Metric; LCSC (none) -> C45783
- D7: footprint Diode_THT:D_DO-41_SOD81_P10.16mm_Horizontal -> Diode_SMD:D_SOD-123; LCSC (none) -> C8598
- FB1: footprint (none) -> Inductor_SMD:L_0805_2012Metric; LCSC (none) -> C21189
- U6: LCSC (none) -> C6186
- U7: footprint (none) -> Package_TO_SOT_SMD:TO-252-3_TabPin2; LCSC (none) -> C58069
Changed lines of the file:
@@
 F 2 "Package_TO_SOT_SMD:SOT-223-3_TabPin2" H 1800 1700 50  0001 C CNN
 F 3 "http://www.advanced-monolithic.com/pdf/ds1117.pdf" H 1900 1250 50  0001 C CNN
+F 4 "C6186" H 1800 1500 50  0001 C CNN "LCSC"
 	1    1800 1500
 	1    0    0    -1
@@
 F 0 "C6" H 2315 1696 50  0000 L CNN
 F 1 "22uF" H 2315 1605 50  0000 L CNN
-F 2 "" H 2238 1500 50  0001 C CNN
+F 2 "Capacitor_SMD:C_0805_2012Metric" H 2238 1500 50  0001 C CNN
 F 3 "~" H 2200 1650 50  0001 C CNN
+F 4 "C45783" H 2200 1650 50  0001 C CNN "LCSC"
 	1    2200 1650
 	1    0    0    -1
@@
 F 0 "C4" H 1415 1696 50  0000 L CNN
 F 1 "22uF" H 1415 1605 50  0000 L CNN
-F 2 "" H 1338 1500 50  0001 C CNN
+F 2 "Capacitor_SMD:C_0805_2012Metric" H 1338 1500 50  0001 C CNN
 F 3 "~" H 1300 1650 50  0001 C CNN
+F 4 "C45783" H 1300 1650 50  0001 C CNN "LCSC"
 	1    1300 1650
 	1    0    0    -1
@@
 F 0 "FB1" V 2313 1500 50  0000 C CNN
 F 1 "Ferrite" V 2404 1500 50  0000 C CNN
-F 2 "" V 2480 1500 50  0001 C CNN
+F 2 "Inductor_SMD:L_0805_2012Metric" V 2480 1500 50  0001 C CNN
 F 3 "~" H 2550 1500 50  0001 C CNN
+F 4 "C21189" H 2550 1500 50  0001 C CNN "LCSC"
 	1    2550 1500
 	0    1    1    0
@@
 F 0 "C8" H 3450 1700 50  0000 L CNN
 F 1 "4.7uF" H 3450 1500 50  0000 L CNN
-F 2 "" H 3488 1450 50  0001 C CNN
+F 2 "Capacitor_SMD:C_0603_1608Metric" H 3488 1450 50  0001 C CNN
 F 3 "~" H 3450 1600 50  0001 C CNN
+F 4 "C19666" H 3450 1600 50  0001 C CNN "LCSC"
 	1    3450 1600
 	1    0    0    -1
@@
 F 0 "C9" H 3700 1700 50  0000 L CNN
 F 1 "100nF" H 3700 1500 50  0000 L CNN
-F 2 "" H 3738 1450 50  0001 C CNN
+F 2 "Capacitor_SMD:C_0603_1608Metric" H 3738 1450 50  0001 C CNN
 F 3 "~" H 3700 1600 50  0001 C CNN
+F 4 "C14663" H 3700 1600 50  0001 C CNN "LCSC"
 	1    3700 1600
 	1    0    0    -1
@@
 F 0 "C10" H 3950 1700 50  0000 L CNN
 F 1 "100nF" H 3950 1500 50  0000 L CNN
-F 2 "" H 3988 1450 50  0001 C CNN
+F 2 "Capacitor_SMD:C_0603_1608Metric" H 3988 1450 50  0001 C CNN
 F 3 "~" H 3950 1600 50  0001 C CNN
+F 4 "C14663" H 3950 1600 50  0001 C CNN "LCSC"
 	1    3950 1600
 	1    0    0    -1
@@
 F 0 "C11" H 4200 1700 50  0000 L CNN
 F 1 "100nF" H 4200 1500 50  0000 L CNN
-F 2 "" H 4238 1450 50  0001 C CNN
+F 2 "Capacitor_SMD:C_0603_1608Metric" H 4238 1450 50  0001 C CNN
 F 3 "~" H 4200 1600 50  0001 C CNN
+F 4 "C14663" H 4200 1600 50  0001 C CNN "LCSC"
 	1    4200 1600
 	1    0    0    -1
@@
 F 0 "C12" H 4450 1700 50  0000 L CNN
 F 1 "100nF" H 4450 1500 50  0000 L CNN
-F 2 "" H 4488 1450 50  0001 C CNN
+F 2 "Capacitor_SMD:C_0603_1608Metric" H 4488 1450 50  0001 C CNN
 F 3 "~" H 4450 1600 50  0001 C CNN
+F 4 "C14663" H 4450 1600 50  0001 C CNN "LCSC"
 	1    4450 1600
 	1    0    0    -1
@@
 F 0 "C13" H 5050 1700 50  0000 L CNN
 F 1 "4.7uF" H 5050 1500 50  0000 L CNN
-F 2 "" H 5088 1450 50  0001 C CNN
+F 2 "Capacitor_SMD:C_0603_1608Metric" H 5088 1450 50  0001 C CNN
 F 3 "~" H 5050 1600 50  0001 C CNN
+F 4 "C19666" H 5050 1600 50  0001 C CNN "LCSC"
 	1    5050 1600
 	1    0    0    -1
@@
 F 0 "C14" H 5300 1700 50  0000 L CNN
 F 1 "100nF" H 5300 1500 50  0000 L CNN
-F 2 "" H 5338 1450 50  0001 C CNN
+F 2 "Capacitor_SMD:C_0603_1608Metric" H 5338 1450 50  0001 C CNN
 F 3 "~" H 5300 1600 50  0001 C CNN
+F 4 "C14663" H 5300 1600 50  0001 C CNN "LCSC"
 	1    5300 1600
 	1    0    0    -1
@@
 F 0 "C15" H 6250 1700 50  0000 L CNN
 F 1 "100nF" H 6250 1500 50  0000 L CNN
-F 2 "" H 6288 1450 50  0001 C CNN
+F 2 "Capacitor_SMD:C_0603_1608Metric" H 6288 1450 50  0001 C CNN
 F 3 "~" H 6250 1600 50  0001 C CNN
+F 4 "C14663" H 6250 1600 50  0001 C CNN "LCSC"
 	1    6250 1600
 	1    0    0    -1
@@
 F 0 "C16" H 7250 1700 50  0000 L CNN
 F 1 "100nF" H 7250 1500 50  0000 L CNN
-F 2 "" H 7288 1450 50  0001 C CNN
+F 2 "Capacitor_SMD:C_0603_1608Metric" H 7288 1450 50  0001 C CNN
 F 3 "~" H 7250 1600 50  0001 C CNN
+F 4 "C14663" H 7250 1600 50  0001 C CNN "LCSC"
 	1    7250 1600
 	1    0    0    -1
@@
 F 0 "U7" H 1900 2300 50  0000 C CNN
 F 1 "L7805" H 1950 2400 50  0000 C CNN
-F 2 "" H 1825 2500 50  0001 L CIN
+F 2 "Package_TO_SOT_SMD:TO-252-3_TabPin2" H 1825 2500 50  0001 L CIN
 F 3 "http://www.st.com/content/ccc/resource/technical/document/datasheet/41/4f/b3/b0/12/d4/47/88/CD00000444.pdf/files/CD00000444.pdf/jcr:content/translations/en.CD00000444.pdf" H 1800 2600 50  0001 C CNN
+F 4 "C58069" H 1800 2650 50  0001 C CNN "LCSC"
 	1    1800 2650
 	1    0    0    -1
@@
 F 0 "C5" H 1300 2900 50  0000 L CNN
 F 1 "4.7uF" H 1300 2700 50  0000 L CNN
-F 2 "" H 1338 2650 50  0001 C CNN
+F 2 "Capacitor_SMD:C_0603_1608Metric" H 1338 2650 50  0001 C CNN
 F 3 "~" H 1300 2800 50  0001 C CNN
+F 4 "C19666" H 1300 2800 50  0001 C CNN "LCSC"
 	1    1300 2800
 	1    0    0    -1
@@
 F 0 "C7" H 2200 2900 50  0000 L CNN
 F 1 "100nF" H 2200 2700 50  0000 L CNN
-F 2 "" H 2238 2650 50  0001 C CNN
+F 2 "Capacitor_SMD:C_0603_1608Metric" H 2238 2650 50  0001 C CNN
 F 3 "~" H 2200 2800 50  0001 C CNN
+F 4 "C14663" H 2200 2800 50  0001 C CNN "LCSC"
 	1    2200 2800
 	1    0    0    -1
@@
 F 0 "D7" H 2450 2433 50  0000 C CNN
 F 1 "1N5819" H 2450 2524 50  0000 C CNN
-F 2 "Diode_THT:D_DO-41_SOD81_P10.16mm_Horizontal" H 2450 2475 50  0001 C CNN
+F 2 "Diode_SMD:D_SOD-123" H 2450 2475 50  0001 C CNN
 F 3 "http://www.vishay.com/docs/88525/1n5817.pdf" H 2450 2650 50  0001 C CNN
+F 4 "C8598" H 2450 2650 50  0001 C CNN "LCSC"
 	1    2450 2650
 	-1   0    0    1

Commit message: finish power board layout first pass
Parts:
- FB1: LCSC C21189 -> e
Changed lines of the file:
@@
 F 2 "Inductor_SMD:L_0805_2012Metric" V 2480 1500 50  0001 C CNN
 F 3 "~" H 2550 1500 50  0001 C CNN
-F 4 "C21189" H 2550 1500 50  0001 C CNN "LCSC"
+F 4 "e" H 2550 1500 50  0001 C CNN "LCSC"
 	1    2550 1500
 	0    1    1    0
