File: hw/MCU_Comms_Control/MCU_Comms_Control.sch (KiCad schematic (older format))
At the start: 33 parts, among them J1 USB_B_Mini, J2 CAN BUS, J3 TO_POWER_BOARD, J4 Mini-Debugging, J5 MULTI, J6 TEMP, SW1 BOOT, SW2 BUTTON, U1 SRV05-4, U2 SN65HVD230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

Commit message: finish new control board revision
Parts:
- removed J5: MULTI, Connector_PinHeader_2.54mm:PinHeader_1x04_P2.54mm_Vertical, symbol Connector_Generic:Conn_01x04
- added D8: FAULT, LED_SMD:LED_0603_1608Metric_Castellated, symbol Device:LED_Small
- added J5: MULTI, Connector_PinHeader_2.54mm:PinHeader_1x06_P2.54mm_Vertical, symbol Connector:Conn_01x06_Male
- added J7: CAN, Connector_PinHeader_2.54mm:PinHeader_1x02_P2.54mm_Vertical, symbol Connector:Conn_01x02_Male
- added JP1: USB PULL, Jumper:SolderJumper-2_P1.3mm_Open_RoundedPad1.0x1.5mm, symbol Jumper:SolderJumper_2_Open
- added R11: 1k5, Resistor_SMD:R_0603_1608Metric, symbol Device:R_Small
- D4, D6: LCSC C72038 -> C72041
- gave numbers to parts that had none: 1
Connections:
- net +3V3: now also J5.1 (Pin_1), JP1.1 (A), R11.2
- net CAN_H: now also J7.1 (Pin_1)
- net CAN_L: now also J7.2 (Pin_2)
- net GND: now also J5.6 (Pin_6)
- net MULTI0: now also U4.56 (PB4), J5.2 (Pin_2); no longer U4.58 (PB6)
- net MULTI1: now also U4.57 (PB5), J5.3 (Pin_3); no longer U4.59 (PB7)
- net USB_D+: now also JP1.2 (B)
- net ~ERROR: now also D8.1 (K)
- net ERR_IN: now reaches U4.25 (PC5)
- net ERR_IN: now also D8.2 (A), R11.1
- new net MULTI2: J5.4 (Pin_4), U4.58 (PB6)
- new net MULTI3: J5.5 (Pin_5), U4.59 (PB7)
Other:
- moved on the sheet: J6
Changed lines of the file:
@@
 Text GLabel 7000 1650 2    39   Input ~ 0
 ~FLASH_CS
-Text GLabel 7000 3550 2    50   Input ~ 0
+Text GLabel 7000 3350 2    50   Input ~ 0
 MULTI0
-Text GLabel 7000 3650 2    50   Input ~ 0
+Text GLabel 7000 3450 2    50   Input ~ 0
 MULTI1
-$Comp
-L Connector_Generic:Conn_01x04 J5
-U 1 1 5FB67D26
-P 2750 5400
-F 0 "J5" H 2668 4975 50  0000 C CNN
-F 1 "MULTI" H 2668 5066 50  0000 C CNN
-F 2 "Connector_PinHeader_2.54mm:PinHeader_1x04_P2.54mm_Vertical" H 2750 5400 50  0001 C CNN
-F 3 "~" H 2750 5400 50  0001 C CNN
-	1    2750 5400
-	-1   0    0    1
-$EndComp
 $Comp
 L power:+3.3V #PWR0134
@@
 L power:GND #PWR0135
 U 1 1 5FB6956E
-P 2950 5500
-F 0 "#PWR0135" H 2950 5250 50  0001 C CNN
-F 1 "GND" V 2955 5372 50  0000 R CNN
-F 2 "" H 2950 5500 50  0001 C CNN
-F 3 "" H 2950 5500 50  0001 C CNN
-	1    2950 5500
+P 2950 5700
+F 0 "#PWR0135" H 2950 5450 50  0001 C CNN
+F 1 "GND" V 2955 5572 50  0000 R CNN
+F 2 "" H 2950 5700 50  0001 C CNN
+F 3 "" H 2950 5700 50  0001 C CNN
+	1    2950 5700
 	1    0    0    -1
 $EndComp
@@
 Text GLabel 2950 5400 2    50   Input ~ 0
 MULTI1
-Wire Wire Line
-	3000 5200 2950 5200
 $Comp
 L Device:R_Small R5
@@
 F 2 "LED_SMD:LED_0603_1608Metric_Castellated" V 3400 1450 50  0001 C CNN
 F 3 "~" V 3400 1450 50  0001 C CNN
-F 4 "C72038" H 3400 1450 50  0001 C CNN "LCSC"
+F 4 "C72041" H 3400 1450 50  0001 C CNN "LCSC"
 	1    3400 1450
 	0    -1   -1   0
@@
 F 2 "LED_SMD:LED_0603_1608Metric_Castellated" V 4200 1450 50  0001 C CNN
 F 3 "~" V 4200 1450 50  0001 C CNN
-F 4 "C72038" H 4200 1450 50  0001 C CNN "LCSC"
+F 4 "C72041" H 4200 1450 50  0001 C CNN "LCSC"
 	1    4200 1450
 	0    -1   -1   0
@@
 L power:GND #PWR01
 U 1 1 5FD220C9
-P 5100 3550
-F 0 "#PWR01" H 5100 3300 50  0001 C CNN
-F 1 "GND" H 5105 3377 50  0000 C CNN
-F 2 "" H 5100 3550 50  0001 C CNN
-F 3 "" H 5100 3550 50  0001 C CNN
-	1    5100 3550
+P 4900 3550
+F 0 "#PWR01" H 4900 3300 50  0001 C CNN
+F 1 "GND" H 4905 3377 50  0000 C CNN
+F 2 "" H 4900 3550 50  0001 C CNN
+F 3 "" H 4900 3550 50  0001 C CNN
+	1    4900 3550
 	1    0    0    -1
 $EndComp
@@
 L Connector:Conn_01x04_Male J6
 U 1 1 5FD31C82
-P 4900 3350
-F 0 "J6" H 5008 3631 50  0000 C CNN
-F 1 "TEMP" H 5008 3540 50  0000 C CNN
-F 2 "Connector_PinHeader_2.54mm:PinHeader_2x02_P2.54mm_Vertical" H 4900 3350 50  0001 C CNN
-F 3 "~" H 4900 3350 50  0001 C CNN
-	1    4900 3350
+P 4700 3350
+F 0 "J6" H 4808 3631 50  0000 C CNN
+F 1 "TEMP" H 4808 3540 50  0000 C CNN
+F 2 "Connector_PinHeader_2.54mm:PinHeader_2x02_P2.54mm_Vertical" H 4700 3350 50  0001 C CNN
+F 3 "~" H 4700 3350 50  0001 C CNN
+	1    4700 3350
 	1    0    0    -1
 $EndComp
@@
 L power:+3.3V #PWR02
 U 1 1 5FD36362
-P 5100 3450
-F 0 "#PWR02" H 5100 3300 50  0001 C CNN
-F 1 "+3.3V" V 5115 3578 50  0000 L CNN
-F 2 "" H 5100 3450 50  0001 C CNN
-F 3 "" H 5100 3450 50  0001 C CNN
-	1    5100 3450
+P 4900 3450
+F 0 "#PWR02" H 4900 3300 50  0001 C CNN
+F 1 "+3.3V" V 4915 3578 50  0000 L CNN
+F 2 "" H 4900 3450 50  0001 C CNN
+F 3 "" H 4900 3450 50  0001 C CNN
+	1    4900 3450
 	0    1    1    0
 $EndComp
@@
 	7400 2750 7000 2750
 $Comp
-L MCU_ST_STM32F3:STM32F303RCTx U?
+L MCU_ST_STM32F3:STM32F303RCTx U4
 U 1 1 5FD72D10
 P 6300 2850
-F 0 "U?" H 6600 1000 50  0000 C CNN
+F 0 "U4" H 6600 1000 50  0000 C CNN
 F 1 "STM32F303RCTx" H 6850 1100 50  0000 C CNN
 F 2 "Package_QFP:LQFP-64_10x10mm_P0.5mm" H 5700 1150 50  0001 R CNN
@@
 Wire Wire Line
 	5300 2200 4850 2200
-Wire Wire Line
-	5600 3250 5100 3250
-Wire Wire Line
-	5600 3350 5100 3350
+Text GLabel 8600 2800 3    50   Input ~ 0
+USB_D+
+$Comp
+L Jumper:SolderJumper_2_Open JP1
+U 1 1 5FDE0DF9
+P 8600 2650
+F 0 "JP1" V 8554 2718 50  0000 L CNN
+F 1 "USB PULL" V 8645 2718 50  0000 L CNN
+F 2 "Jumper:SolderJumper-2_P1.3mm_Open_RoundedPad1.0x1.5mm" H 8600 2650 50  0001 C CNN
+F 3 "~" H 8600 2650 50  0001 C CNN
+	1    8600 2650
+	0    1    1    0
+$EndComp
+$Comp
+L power:+3V3 #PWR04
+U 1 1 5FDE19FA
+P 8600 2500
+F 0 "#PWR04" H 8600 2350 50  0001 C CNN
+F 1 "+3V3" H 8615 2673 50  0000 C CNN
+F 2 "" H 8600 2500 50  0001 C CNN
+F 3 "" H 8600 2500 50  0001 C CNN
+	1    8600 2500
+	1    0    0    -1
+$EndComp
+Text GLabel 7000 3550 2    50   Input ~ 0
+MULTI2
+Text GLabel 7000 3650 2    50   Input ~ 0
+MULTI3
+Text GLabel 2950 5500 2    50   Input ~ 0
+MULTI2
+Text GLabel 2950 5600 2    50   Input ~ 0
+MULTI3
+$Comp
+L Connector:Conn_01x06_Male J5
+U 1 1 5FDEA331
+P 2650 5400
+F 0 "J5" H 2758 5781 50  0000 C CNN
+F 1 "MULTI" H 2758 5690 50  0000 C CNN
+F 2 "Connector_PinHeader_2.54mm:PinHeader_1x06_P2.54mm_Vertical" H 2650 5400 50  0001 C CNN
+F 3 "~" H 2650 5400 50  0001 C CNN
+	1    2650 5400
+	1    0    0    -1
+$EndComp
+Wire Wire Line
+	2950 5700 2850 5700
+Wire Wire Line
+	2950 5500 2850 5500
+Wire Wire Line
+	2850 5600 2950 5600
+Wire Wire Line
+	2950 5400 2850 5400
+Wire Wire Line
+	2950 5300 2850 5300
+Wire Wire Line
+	2850 5200 3000 5200
+$Comp
+L Connector:Conn_01x02_Male J7
+U 1 1 5FE0DA52
+P 5900 5700
+F 0 "J7" H 5872 5674 50  0000 R CNN
+F 1 "CAN" H 5872 5583 50  0000 R CNN
+F 2 "Connector_PinHeader_2.54mm:PinHeader_1x02_P2.54mm_Vertical" H 5900 5700 50  0001 C CNN
+F 3 "~" H 5900 5700 50  0001 C CNN
+	1    5900 5700
+	-1   0    0    -1
+$EndComp
+Text GLabel 5700 5700 0    50   Input ~ 0
+CAN_H
+Text GLabel 5700 5800 0    50   Input ~ 0
+CAN_L
+Text GLabel 8050 5600 3    50   Input ~ 10
+~ERROR
+Text GLabel 8050 5250 2    50   Input ~ 0
+ERR_IN
+$Comp
+L Device:R_Small R11
+U 1 1 5FE42D95
+P 8050 5100
+F 0 "R11" V 7854 5100 50  0000 C CNN
+F 1 "1k5" V 7945 5100 50  0000 C CNN
+F 2 "Resistor_SMD:R_0603_1608Metric" H 8050 5100 50  0001 C CNN
+F 3 "~" H 8050 5100 50  0001 C CNN
+F 4 "C22843" H 8050 5100 50  0001 C CNN "LCSC"
+	1    8050 5100
+	-1   0    0    1
+$EndComp
+$Comp
+L power:+3V3 #PWR03
+U 1 1 5FE455CF
+P 8050 5000
+F 0 "#PWR03" H 8050 4850 50  0001 C CNN
+F 1 "+3V3" H 8065 5173 50  0000 C CNN
+F 2 "" H 8050 5000 50  0001 C CNN
+F 3 "" H 8050 5000 50  0001 C CNN
+	1    8050 5000
+	1    0    0    -1
+$EndComp
+Text GLabel 5600 3450 0    50   Input ~ 0
+ERR_IN
+Wire Wire Line
+	4900 3350 5600 3350
+Wire Wire Line
+	4900 3250 5600 3250
+$Comp
+L Device:LED_Small D8
+U 1 1 5FE6FA92
+P 8050 5450
+F 0 "D8" V 8096 5380 50  0000 R CNN
+F 1 "FAULT" V 8005 5380 50  0000 R CNN
+F 2 "LED_SMD:LED_0603_1608Metric_Castellated" V 8050 5450 50  0001 C CNN
+F 3 "~" V 8050 5450 50  0001 C CNN
+F 4 "C2286" H 8050 5450 50  0001 C CNN "LCSC"
+	1    8050 5450
+	0    -1   -1   0
+$EndComp
+Wire Wire Line
+	8050 5600 8050 5550
+Wire Wire Line
+	8050 5200 8050 5350
 $EndSCHEMATC
