File: hw/MCU_Comms_Control/MCU_Comms_Control.sch (KiCad schematic (older format))
At the start: 37 parts, among them J1 USB_B_Mini, J2 CAN BUS, J3 TO_POWER_BOARD, J4 Mini-Debugging, J5 MULTI, J6 TEMP, J7 CAN, SW1 BOOT, SW2 BUTTON, U1 SRV05-4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

Commit message: fix boot0 resistor
Connections:
- net +3V3: now also SW1.2 (B); no longer R1.2
- net GND: now also R1.1; no longer SW1.2 (B)
- net ~BOOT: now also R1.2; no longer R1.1
Other:
- note added: "Changed from\npull-up to pull-down\n"
- moved on the sheet: R1
Changed lines of the file:
@@
 	1    0    0    1
 $EndComp
-$Comp
-L Device:R_Small R1
-U 1 1 5FB977A0
-P 5300 1100
-F 0 "R1" H 5241 1054 50  0000 R CNN
-F 1 "4k7" H 5241 1145 50  0000 R CNN
-F 2 "Resistor_SMD:R_0603_1608Metric" H 5300 1100 50  0001 C CNN
-F 3 "~" H 5300 1100 50  0001 C CNN
-F 4 "C23162" H 5300 1100 50  0001 C CNN "LCSC"
-	1    5300 1100
-	1    0    0    1
-$EndComp
-Wire Wire Line
-	5600 1450 5300 1450
-Wire Wire Line
-	5300 1450 5300 1200
+Wire Wire Line
+	5600 1450 5500 1450
 Wire Wire Line
 	5600 1250 5550 1250
@@
 Wire Wire Line
 	5550 950  5450 950
-Wire Wire Line
-	5300 950  5300 1000
 $Comp
 L power:+3V3 #PWR0120
@@
 Wire Wire Line
 	5450 850  5450 950
-Connection ~ 5450 950
-Wire Wire Line
-	5450 950  5300 950
 Text GLabel 5550 1250 0    39   Input ~ 0
 ~RESET
@@
 $EndComp
 Wire Wire Line
-	3750 2450 3700 2450
-Wire Wire Line
-	3700 2450 3700 2100
-Wire Wire Line
 	3700 2100 3650 2100
-Connection ~ 3700 2450
-Wire Wire Line
-	3700 2450 3650 2450
 Text GLabel 7000 2950 2    50   Input ~ 0
 CURR_U
@@
 Wire Wire Line
 	8050 5200 8050 5350
+$Comp
+L Device:R_Small R1
+U 1 1 5FB977A0
+P 5500 1550
+F 0 "R1" H 5441 1504 50  0000 R CNN
+F 1 "4k7" H 5441 1595 50  0000 R CNN
+F 2 "Resistor_SMD:R_0603_1608Metric" H 5500 1550 50  0001 C CNN
+F 3 "~" H 5500 1550 50  0001 C CNN
+F 4 "C23162" H 5500 1550 50  0001 C CNN "LCSC"
+	1    5500 1550
+	1    0    0    1
+$EndComp
+Connection ~ 5500 1450
+Wire Wire Line
+	5500 1450 5300 1450
+$Comp
+L power:GND #PWR?
+U 1 1 6001C778
+P 5500 1650
+F 0 "#PWR?" H 5500 1400 50  0001 C CNN
+F 1 "GND" H 5505 1477 50  0000 C CNN
+F 2 "" H 5500 1650 50  0001 C CNN
+F 3 "" H 5500 1650 50  0001 C CNN
+	1    5500 1650
+	1    0    0    -1
+$EndComp
+Text Notes 4600 1700 0    50   ~ 10
+Changed from\npull-up to pull-down\n
+Wire Wire Line
+	3650 2450 3750 2450
+$Comp
+L power:+3V3 #PWR?
+U 1 1 60024A22
+P 3700 2100
+F 0 "#PWR?" H 3700 1950 50  0001 C CNN
+F 1 "+3V3" V 3715 2228 50  0000 L CNN
+F 2 "" H 3700 2100 50  0001 C CNN
+F 3 "" H 3700 2100 50  0001 C CNN
+	1    3700 2100
+	0    1    1    0
+$EndComp
 $EndSCHEMATC

Commit message: tag wrong crystal footprint
Other:
- note added: "FIXME\nWRONG FOOTPRINT"
Changed lines of the file:
@@
 	0    1    1    0
 $EndComp
+Text Notes 5300 2750 1    50   ~ 10
+FIXME\nWRONG FOOTPRINT
 $EndSCHEMATC

Commit message: mini-fit (CAN) connector hole size from 1.4 to 1.8mm diameter and add silkscreen labels for the debugger pins
Parts:
- J1: symbol Connector:USB_B_Mini -> MCU_Comms_Control-rescue:USB_B_Mini-Connector
Changed lines of the file:
@@
 Pull-up resistor for\nfull-speed identification
 $Comp
-L Connector:USB_B_Mini J1
+L MCU_Comms_Control-rescue:USB_B_Mini-Connector J1
 U 1 1 5FBAAB5E
 P 900 6800
